File: Adapter_RCB_F9T.kicad_pcb (KiCad board)
At the start: 4 copper layers, 32 x 83 mm, 48 parts, among them J1 USB_B_Micro, J2 Conn_01x04, J41 RCB_F9T, J51 Conn_Coaxial, J61 Conn_Coaxial, U11 XC6206PxxxMR, U21 LM27761, U31 CP2102-GMR-xQFN28, U51 BUF602xDBV, U61 BUF602xDBV

Commit message: fix RCB-F9T NRST issue and move FB41 further away from mounting hole
Parts:
- removed R41: 4k7, Resistor_SMD:R_0402_1005Metric
- added JP41: SolderJumper_2_Open, Jumper:SolderJumper-2_P1.3mm_Open_RoundedPad1.0x1.5mm, B.Cu at (77.0, 92.5)
- moved FB41 2.00 mm to (83.0, 94.0)
Routing:
- net Net-(J41-V_ANT): track 9.66 -> 11.4 mm
- net GND: track 52.4 -> 52.3 mm, vias 230 -> 229
Other:
- board text added: "RCB-F9T Adapter r2"
- board text removed: "RCB-F9T Adapter r1"
